File: Apple2Uthernet.kicad_pcb (KiCad board)
At the start: 2 copper layers, 100 x 69.8 mm, 69 parts, among them J1 Apple II Bus Card Edge, J2 RJ45_LED_Shielded, U1 74LS139, U2 74LS245, U3 W5100, U4 NCP1117-3.3_SOT223, U5 74LVC1G07, U6 74LVC1G17, U7 74LVC1G17, U8 74LVC1G17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

Commit message: Updated PCB Layout to accomodate Adafruit Panel Mount Ethernet Extension Cable (PN 909). Made the board more compact. Updated project to render 3D models properly. Added edge rails/fiducials as per https://jlcpcb.com/help/article/48-How-to-add-edge-rails%2Ffiducials-for-PCB-assembly-order Very little should need to be moved around or fixing.
Parts:
- added REF1: Fiducial_1mm_Mask3mm, Fiducial:Fiducial_1mm_Mask3mm, F.Cu at (203.5, 128.4)
- added REF2: Fiducial_1mm_Mask3mm, Fiducial:Fiducial_1mm_Mask3mm, F.Cu at (259.2, 67.2)
- D1: footprint Diode_SMD:D_SOD-323F -> Diode_SMD:D_SOD-523
- D8: value POWERLED -> POWER LED
- moved FB3 97.6 mm to (256.5, 72.9), turned to 90 degrees
- moved C10 97.5 mm to (252.3, 73.5)
- moved C11 96.2 mm to (254.5, 72.9)
- moved C9 94.1 mm to (256.5, 79.3)
- moved C16 90.8 mm to (220.2, 86.1), turned to 0 degrees
- moved C17 90.8 mm to (220.2, 89.4), turned to 0 degrees
- moved C4 90.5 mm to (213.4, 82.3)
- moved J2 90.5 mm to (200.2, 78.2)
- moved R14 90.5 mm to (213.4, 80.2)
- moved R15 90.5 mm to (213.4, 78.2)
- moved R6 90.5 mm to (213.4, 76.1)
- moved R7 90.5 mm to (213.4, 74.1)
- moved C3 90.5 mm to (220.1, 74.1)
- moved R3 90.5 mm to (197.9, 68.7)
- moved R4 90.5 mm to (197.9, 87.6)
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Routing:
- net Earth: track 358.4 -> 196.3 mm
- net /~{IRQ}: track 17.6 -> 63.8 mm
- net +5V: track 115.2 -> 150.1 mm
- net +3.3V: track 166.3 -> 132.9 mm, vias 5 -> 4
- net /W5100_INT: track 48.8 -> 18.0 mm, vias 0 -> 2
- net GNDA: track 113.1 -> 87.0 mm
- net /W5100_FDXLED: track 101.8 -> 78.8 mm
- net /W5100_LINKLED: track 99.9 -> 76.9 mm
- net /W5100_A1: track 49.7 -> 71.8 mm
- net /W5100_A0: track 51.7 -> 72.7 mm
- net +3V3A: track 136.9 -> 156.0 mm
- net /W5100_TXLED: track 63.0 -> 45.0 mm
- net /W5100_COLLED: track 55.1 -> 37.1 mm
- net /W5100_SPDLED: track 46.4 -> 28.4 mm
- net /W5100_RXLED: track 59.0 -> 41.0 mm
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Other:
- board size 100 x 69.8 mm -> 79.8 x 69.8 mm
- board text added: "Slot 2 Cutout for Adafruit Panel Mount Ethernet Extension Cable https://www.adafru.it/P909"
