File: Apple2Uthernet.kicad_sch (KiCad schematic)
At the start: 70 parts, among them J1 Apple II Bus Card Edge, J2 RJ45_LED_Shielded, U1 74LS139, U2 74LS245, U3 W5100, U4 NCP1117-3.3_SOT223, U5 74LVC1G07, U6 74LVC1G17, U7 74LVC1G17, U8 74LVC1G17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

Commit message: Updated PCB Layout to accomodate Adafruit Panel Mount Ethernet Extension Cable (PN 909). Made the board more compact. Updated project to render 3D models properly. Added edge rails/fiducials as per https://jlcpcb.com/help/article/48-How-to-add-edge-rails%2Ffiducials-for-PCB-assembly-order Very little should need to be moved around or fixing.
Parts:
- added REF1, REF2: Fiducial_1mm_Mask3mm, Fiducial:Fiducial_1mm_Mask3mm, symbol Mechanical:Fiducial
- C1, C2: Digi-Key_PN 13-CC0805JRNPO9BN130CT-ND -> (none); PN_DigiKey (none) -> 13-CC0805JRNPO9BN130CT-ND
- C10, C7, C8, C9: Digi-Key_PN 399-3824-1-ND -> (none); PN_DigiKey (none) -> 399-3824-1-ND
- C11: Digi-Key_PN 1276-2984-1-ND -> (none); PN_DigiKey (none) -> 1276-2984-1-ND
- C12, C13, C14, C15, C16, C17, C18, C19, C20, C23, C26, C27, C28, C3, C4, C5: Digi-Key_PN 1276-1003-1-ND -> (none); PN_DigiKey (none) -> 1276-1003-1-ND
- C21: Digi-Key_PN 1276-2605-1-ND -> (none); PN_DigiKey (none) -> 1276-2605-1-ND
- C22: Digi-Key_PN 1276-1014-1-ND -> (none); PN_DigiKey (none) -> 1276-1014-1-ND
- C24: Digi-Key_PN 1276-CL21B106KAYQNNECT-ND -> (none); PN_DigiKey (none) -> 1276-CL21B106KAYQNNECT-ND
- C25: Digi-Key_PN 1276-CL21A226MAYNNNECT-ND -> (none); PN_DigiKey (none) -> 1276-CL21A226MAYNNNECT-ND
- C6: Digi-Key_PN 399-8284-1-ND -> (none); LCSC C1952847 -> C1954959; PN_DigiKey (none) -> 399-8284-1-ND
- D1: footprint Diode_SMD:D_SOD-323F -> Diode_SMD:D_SOD-523; Digi-Key_PN 1N914BWSCT-ND -> (none); LCSC C258181 -> C2836064; PN_DigiKey (none) -> 1N914BWSCT-ND
- D2, D3, D4, D5, D6, D7: Digi-Key_PN 754-1127-1-ND -> (none); PN_DigiKey (none) -> 754-1127-1-ND
- D8: value POWERLED -> POWER LED; Digi-Key_PN 754-1127-1-ND -> (none); PN_DigiKey (none) -> 754-1127-1-ND
- FB1, FB2: Digi-Key_PN 445-6391-1-ND -> (none); PN_DigiKey (none) -> 445-6391-1-ND
- FB3: Digi-Key_PN 445-6391-1-ND -> (none); PN_DigiKey (none) -> 445-6391-1-ND; PN_Mouser (none) -> 810-MLZ2012A1R0WT000
- J2: Digi-Key_PN MJ3230-88-GG-2 -> (none); PN_DigiKey (none) -> MJ3230-88-GG-2
- R1: Digi-Key_PN 10-ERJ-P06F1004VCT-ND -> (none); PN_DigiKey (none) -> 10-ERJ-P06F1004VCT-ND
- R10, R11, R12, R2, R5: Digi-Key_PN P590CCT-ND -> (none); PN_DigiKey (none) -> P590CCT-ND
- R13: Digi-Key_PN P590CCT-ND -> (none); PN_DigiKey (none) -> P590CCT-ND; PN_Mouser (none) -> 667-ERJ-6ENF5900V
- R14, R15, R17, R6, R7: Digi-Key_PN 541-49.9TCT-ND -> (none); LCSC C4088942 -> C204544; PN_DigiKey (none) -> 541-49.9TCT-ND
- R16, R19: Digi-Key_PN P16073CT-ND -> (none); PN_DigiKey (none) -> P16073CT-ND
- R18: Digi-Key_PN P1.43KCCT-ND -> (none); LCSC C2077366 -> C101474; PN_DigiKey (none) -> P1.43KCCT-ND
- R3, R4: Digi-Key_PN P330CCT-ND -> (none); PN_DigiKey (none) -> P330CCT-ND
- R8: Digi-Key_PN 311-300CRCT-ND -> (none); PN_DigiKey (none) -> 311-300CRCT-ND
- R9: Digi-Key_PN 13-RC0805FR-7W12KL-ND -> (none); LCSC C7038301 -> C408920; PN_DigiKey (none) -> 13-RC0805FR-7W12KL-ND
- U1: Digi-Key_PN 2156-DM74LS139SJ-ND -> (none); PN_DigiKey (none) -> 2156-DM74LS139SJ-ND
- U2: Digi-Key_PN 296-3677-1-ND -> (none); PN_DigiKey (none) -> 296-3677-1-ND
- U3: Digi-Key_PN 1278-1002-ND -> (none); PN_DigiKey (none) -> 1278-1002-ND
- U4: Digi-Key_PN NCP1117ST33T3GOSCT-ND -> (none); PN_DigiKey (none) -> NCP1117ST33T3GOSCT-ND
- U5: Digi-Key_PN 296-8485-1-ND -> (none); PN_DigiKey (none) -> 296-8485-1-ND
- U6, U7, U8: Digi-Key_PN 296-11933-1-ND -> (none); PN_DigiKey (none) -> 296-11933-1-ND
- Y1: Digi-Key_PN CTX652CT-ND -> (none); LCSC C2961981 -> C252362; PN_DigiKey (none) -> CTX652CT-ND

Commit message: Updated Fiducial rails; Changed 1 resistor due to stocking issues.
Parts:
- R18: LCSC C101474 -> C336837
Changed lines of the file:
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@@
       (effects (font (size 1.27 1.27)) hide)
     )
-    (property "LCSC" "C101474" (id 6) (at 281.94 104.14 0)
+    (property "LCSC" "C336837" (id 6) (at 281.94 104.14 0)
       (effects (font (size 1.27 1.27)) hide)
     )
